File: sensor_gnuiiium/sensor_gnuiiium.kicad_pcb (KiCad board)
At the start: 2 copper layers, 75 x 40 mm, 37 parts, among them J1 jumper, J10 Conn_01x10_Male, J2 jumper, J3 jumper, J4 jumper, J5 jumper, J6 jumper, J7 jumper, J8 jumper, U1 qrd111x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

Commit message: generated gerber files
Other:
- board text added: "solsticio"
Changed lines of the file:
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@@
       (outputformat 1)
       (mirror false)
-      (drillshape 1)
+      (drillshape 0)
       (scaleselection 1)
-      (outputdirectory "")
+      (outputdirectory "gerbers/")
     )
   )
@@
   (gr_line (start 172.5 116.3066) (end 179.375 116.3066) (layer "User.1") (width 0.1))
   (gr_line (start 179.3494 123.2916) (end 179.3494 30.015) (layer "User.1") (width 0.1))
+  (gr_text "solsticio" (at 203.2 83.82) (layer "F.Cu")
+    (effects (font (size 1.5 1.5) (thickness 0.3)))
+  )
   (segment (start 188.468 101.6) (end 188.468 98.425) (width 1.27) (layer "F.Cu") (net 1))
   (segment (start 197.256 98.45) (end 193.929 95.123) (width 1.27) (layer "F.Cu") (net 1))

Commit message: Flipped the sensors
Parts:
- U1, U2, U3, U4, U5, U6, U7, U8: moved to B.Cu
- moved U1 66.1 mm to (212.3, 116.2), turned to 0 degrees
- moved U8 63.9 mm to (147.3, 116.2), turned to 0 degrees
- moved U7 48.9 mm to (154.8, 116.2), turned to 0 degrees
- moved U2 48.6 mm to (203.6, 116.2), turned to 0 degrees
- moved U6 31.4 mm to (163.6, 116.2), turned to 0 degrees
- moved U3 31.1 mm to (194.8, 116.2), turned to 0 degrees
- moved U5 13.9 mm to (172.3, 116.2), turned to 0 degrees
- moved U4 13.6 mm to (186.1, 116.2), turned to 0 degrees
