File: sensor_gnuiiium/sensor_gnuiiium.kicad_sch (KiCad schematic)
At the start: 35 parts, among them J1 jumper, J10 Conn_01x10_Male, J2 jumper, J3 jumper, J4 jumper, J5 jumper, J6 jumper, J7 jumper, J8 jumper, U1 qrd111x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

Commit message: changed to smd version
Parts:
- J10: footprint (none) -> Connector_PinSocket_2.54mm:PinSocket_1x10_P2.54mm_Vertical
- R1, R10, R11, R12, R13, R14, R15, R16, R2, R3, R4, R5, R6, R7, R8, R9: footprint Resistor_THT:R_Axial_DIN0207_L6.3mm_D2.5mm_P10.16mm_Horizontal -> Resistor_SMD:R_0805_2012Metric_Pad1.20x1.40mm_HandSolder
